Commit message: Fix configs. Now working!

File: urdf/backpack_2d.urdf (robot description, URDF)
Before this commit: robot cartographer_backpack_2d, 1 links, 0 joints
Links:
- added link laser
Joints:
- added joint laser_link_joint: type fixed, parent base_link, child laser, origin xyz=0 0 0

Commit message: Add navigation.

File: urdf/backpack_2d.urdf (robot description, URDF)
Before this commit: robot cartographer_backpack_2d, 2 links, 1 joints
Joints:
- joint laser_link_joint: origin xyz=0 0 0 -> xyz=0 0 0 rpy=0 0 3.14

Commit message: Start implementing Complete Coverage algorithm.

File: urdf/backpack_2d.urdf (robot description, URDF)
Before this commit: robot cartographer_backpack_2d, 2 links, 1 joints
Joints:
- joint laser_link_joint: origin xyz=0 0 0 rpy=0 0 3.14 -> xyz=0 0 0 rpy=0 0 0
